File: ampli tda/ampli tda.kicad_pcb (KiCad board)
At the start: 2 copper layers, 85 x 50 mm, 23 parts, among them J1 Barrel_Jack, J2 Conn_01x03_Pin, U1 TDA2003

Commit message: REV 0.2
Update
Parts:
- added C7: 100nF, Capacitor_THT:C_Disc_D7.5mm_W2.5mm_P5.00mm, F.Cu at (176.0, 58.2)
Connections:
- RV1 pad 3: GND -> Net-(C7-Pad1)
Routing:
- net Net-(C7-Pad1): track 0.00 -> 12.5 mm
Other:
- board text added: "REV 0.2"
- board text removed: "REV 0.1"
